File: design/design.kicad_sch (KiCad schematic)
At the start: 1 part, among them U1 MCIMX6XxxVN

Commit message: initial ldo
Signed-off-by: Zbigniew Opiol <zbigniew.opiol@tbs-biometrics.com>
Parts:
- removed U1: MCIMX6XxxVN, zbop:LFBGA400, symbol zbop:MCIMX6XxxVN
Other:
- added sheet power (power.kicad_sch)
