File: design/design.kicad_sch (KiCad schematic)
At the start: 0 parts

Commit message: sch: power tree: possibly finished pmic
Signed-off-by: Zbigniew Opiol <zbigniew.opiol@tbs-biometrics.com>
Other:
- sheet power ports: added INTB, ONKEY, PWRON, RESETBMCU, STNDBY, VLDO1, Varm, Vddr, Vrefddr, Vsnvs, Vsoc, WDI; removed none

Commit message: sch: ddr3 in progress
Signed-off-by: Zbigniew Opiol <zbigniew.opiol@tbs-biometrics.com>
Other:
- added sheet CPU (cpu.kicad_sch)
- added sheet DDR3 (ddr3.kicad_sch)
- added sheet pwr (pwr.kicad_sch)
