File: design/power.kicad_sch (KiCad schematic)
At the start: 25 parts

Commit message: sch: power tree: possibly finished pmic
Signed-off-by: Zbigniew Opiol <zbigniew.opiol@tbs-biometrics.com>
Parts:
- added C? (x6): 1uF, Capacitor_SMD:C_0805_2012Metric_Pad1.18x1.45mm_HandSolder, symbol Device:C_Small
- added C? (x6): 10u, Capacitor_SMD:C_0805_2012Metric_Pad1.18x1.45mm_HandSolder, symbol Device:C_Small
- added C? (x3): 4u7, Capacitor_SMD:C_0805_2012Metric_Pad1.18x1.45mm_HandSolder, symbol Device:C_Small
- added D?: RED, LED_SMD:LED_0805_2012Metric_Pad1.15x1.40mm_HandSolder, symbol Device:LED
- added J? (x6): Conn_01x02, symbol Connector_Generic:Conn_01x02
- added J?: Conn_01x04, symbol Connector_Generic:Conn_01x04
- added J?: Conn_01x03, symbol Connector_Generic:Conn_01x03
- added L? (x3): 1uH, Inductor_SMD:L_0201_0603Metric_Pad0.64x0.40mm_HandSolder, symbol Device:L_Small
- added R?: 47R, Resistor_SMD:R_0805_2012Metric_Pad1.20x1.40mm_HandSolder, symbol Device:R_US
- added R?: 10k, Resistor_SMD:R_0805_2012Metric_Pad1.20x1.40mm_HandSolder, symbol Device:R_US
- added TP? (x4): TestPoint, symbol Connector:TestPoint
Connections:
- net GND: now also U?.5 (VDDOTP), C?.2, C?.2, C?.2, C?.2, C?.2, C?.2, C?.2, C?.2, C?.2, C?.2, C?.2, C?.2, C?.2, C?.2, C?.2, J?.3 (Pin_3), J?.4 (Pin_4)
- net ONKEY: now also TP?.1
- net PWRON: now also TP?.1
- net STNDBY: now also TP?.1
- net Vsys: now also R?.2
- net WDI: now also TP?.1
- net RESETBMCU: now reaches U?.10 (RESETBMCU)
- net VLDO3: now reaches U?.12 (VLDO3)
- net VLDO3: now also C?.1, J?.3 (Pin_3)
- net at U?.13 (SW3LX): now also L?.1
- net at U?.15 (SW3FB): now also C?.1, C?.1, J?.2 (Pin_2), L?.2
- net Vrefin: now reaches U?.16 (SW2FB)
- net Vrefin: now also U?.22 (VINREFDDR), C?.1, C?.1, J?.2 (Pin_2), L?.2
- net at U?.18 (SW2LX): now also L?.1
- net VLDO2: now reaches U?.19 (VLDO2)
- net VLDO2: now also C?.1, J?.2 (Pin_2)
- net at U?.21 (VREFDDR): now also C?.1, J?.2 (Pin_2)
- net at U?.23 (VDIG): now also C?.1
- net at U?.24 (VCORE): now also C?.1
- net at U?.25 (SW1LX): now also L?.1
- net at U?.27 (SW1FB): now also C?.1, C?.1, J?.2 (Pin_2), L?.2
- net VLDO1: now reaches U?.29 (VLDO1)
- net VLDO1: now also C?.1, J?.1 (Pin_1)
- net at U?.30 (VSNVS): now also C?.1, J?.2 (Pin_2)
- net at U?.32 (THM): now also J?.2 (Pin_2), R?.2
- net at U?.33 (VBAT1): now also U?.34 (VBAT2), J?.1 (Pin_1)
- net at U?.37 (VBUSIN): now also J?.2 (Pin_2)
- net at U?.38 (INT2P7): now also C?.1, C?.1, R?.1
- net at U?.39 (USBPHY): now also J?.1 (Pin_1)
- net at U?.40 (CHGB): now also D?.1 (K)
- net INTB: now reaches U?.9 (INTB)
- new net: D?.2 (A), R?.1
- new net Varm: J?.1 (Pin_1)
- new net Vddr: J?.1 (Pin_1)
- new net Vrefddr: J?.1 (Pin_1)
- new net Vsnvs: J?.1 (Pin_1)
- new net Vsoc: J?.1 (Pin_1)
- no-connect marks 2 -> 0
Other:
- note added: "1.4V"
- note added: "3.7V Li-Ion 10k thermistor"

Commit message: sch: ddr3 in progress
Signed-off-by: Zbigniew Opiol <zbigniew.opiol@tbs-biometrics.com>
Parts:
- gave numbers to parts that had none: 58
